File: MDcir_v0.2.1/MD_v0.2.1.sch (KiCad schematic (older format))
At the start: 63 parts, among them IC1 ADUM1310, IC2 A3941, IC3 ACS715, J1 RJ45, J2 RJ45, P1 XA_5Pin, P2 ST-LINK, P3 SEL_5V, P4 MOTOR, P5 SEL_5V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

Commit message: 
Parts:
- U3: symbol 7805 -> 7805-RESCUE-MD_v0.2.1
Changed lines of the file:
@@
 $EndComp
 $Comp
-L 7805 U3
+L 7805-RESCUE-MD_v0.2.1 U3
 U 1 1 58D06069
 P 7850 1450
